File: ESP32 Audio Player/ESP32 Audio Player.kicad_pcb (KiCad board)
At the start: 2 copper layers, 8 parts, among them SW1 SW_Push, SW2 SW_Push, SW3 SW_Push, U1 TP4056, U2 OLED

Commit message: Completed main firmware
Parts:
- AMP1, MCU1, U1: moved to B.Cu
- SD1: footprint Extras:SD Card Reader -> Micro SD Card Reader:MODULE_MICROSD_SPI_OR_SDIO_CARD; moved to B.Cu
- moved U1 148.6 mm to (79.5, 44.0), turned to 0 degrees
- moved SD1 143.0 mm to (73.1, 74.0), turned to -90 degrees
- moved SW3 92.7 mm to (127.5, 91.0)
- moved U2 90.1 mm to (105.5, 65.0)
- moved SW2 87.8 mm to (105.0, 91.0)
- moved SW1 82.8 mm to (81.0, 91.0)
- moved MCU1 75.7 mm to (89.9, 44.7), turned to -90 degrees
- moved AMP1 64.7 mm to (133.0, 56.0), turned to 0 degrees
Connections:
- MCU1 pad 1: unconnected-(MCU1-3V3-Pad1) -> 3V3
- SD1 pad 1: GND -> 3V3
- SD1 pad 2: 5V -> Net-(MCU1-D5)
- SD1 pad 6: Net-(MCU1-D5) -> GND
Routing:
- net (no net): track 4.54 -> 0.00 mm, vias 1 -> 0

Commit message: Completed PCB
Parts:
- Battery Charger: renamed from U1
- moved AMP1 3.58 mm to (129.4, 56.0)
- renumbered MCU1 to ESP32
Routing:
- net GND: track 0.00 -> 194.7 mm
- net Net-(MCU1-D23): track 0.00 -> 116.6 mm, vias 0 -> 4
- net 5V: track 0.00 -> 75.7 mm
- net Net-(MCU1-D18): track 0.00 -> 65.8 mm, vias 0 -> 1
- net Net-(MCU1-D19): track 0.00 -> 63.9 mm, vias 0 -> 1
- net Net-(MCU1-D5): track 0.00 -> 63.1 mm, vias 0 -> 3
- net Net-(AMP1-LRC): track 0.00 -> 55.8 mm, vias 0 -> 2
- net Net-(AMP1-BCLK): track 0.00 -> 55.1 mm, vias 0 -> 2
- net Net-(AMP1-DIN): track 0.00 -> 54.3 mm, vias 0 -> 2
- net Net-(MCU1-D34): track 0.00 -> 48.6 mm, vias 0 -> 1
- net Net-(MCU1-VN): track 0.00 -> 45.8 mm
- net 3V3: track 0.00 -> 41.0 mm, vias 0 -> 1
- net Net-(MCU1-VP): track 0.00 -> 39.4 mm
- net SDA: track 0.00 -> 26.2 mm, vias 0 -> 1
- net SCL: track 0.00 -> 21.7 mm
Other:
- board outline added: 75.5 x 72 mm
- board text added: "15"
- board text added: "3V3"
- board text added: "5V"
- board text added: "GND"
- board text added: "Original Creator: theNeonTerminal https://github.com/theNeonTerminal https://github.com/theNeonTerminal/ESP32-Audio-Player"
- board text added: "SCL"
- board text added: "SDA"

Commit message: Added README and Updated PCB
Parts:
- removed AMP1: adafruit-MAX98357, MAX98357A:adafruit-MAX98357
- added DAC1: PCM5102a, PCM5102a:GY-PCM5102, B.Cu at (129.5, 47.5)
- U1: renamed from Battery Charger
- renumbered ESP32 to MCU1
Routing:
- net GND: track 194.7 -> 227.4 mm
- net 5V: track 75.7 -> 88.7 mm
- net Net-(DAC1-BCK): track 55.1 -> 45.7 mm, vias 2 -> 1
- net Net-(DAC1-DIN): track 54.3 -> 46.3 mm, vias 2 -> 3
- net Net-(MCU1-D23): track 116.6 -> 112.0 mm
- net Net-(DAC1-LCK): track 55.8 -> 53.8 mm

Commit message: Added gerber files
Routing:
- added copper zone on B.Cu, net GND
- added copper zone on F.Cu, net GND
Changed lines of the file:
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@@
 			(outputformat 1)
 			(mirror no)
-			(drillshape 1)
+			(drillshape 0)
 			(scaleselection 1)
-			(outputdirectory "")
+			(outputdirectory "ESP32 Audio Player/")
 		)
 	)
@@
 	)
 	(segment
-		(start 73 68)
-		(end 74.5 68)
+		(start 94.5 37)
+		(end 94.5 34.38)
 		(width 0.5)
 		(layer "B.Cu")
@@
 	)
 	(segment
-		(start 94.5 37)
-		(end 94.5 34.38)
+		(start 73 68)
+		(end 71 66)
 		(width 0.5)
 		(layer "B.Cu")
@@
 	)
 	(segment
-		(start 71 66)
+		(start 74.5 68)
 		(end 73 68)
 		(width 0.5)
@@
 		(net "Net-(MCU1-D18)")
 	)
+	(zone
+		(net "GND")
+		(layer "F.Cu")
+		(hatch edge 0.5)
+		(connect_pads
+			(clearance 0.5)
+		)
+		(min_thickness 0.25)
+		(fill yes
+			(thermal_gap 0.5)
+			(thermal_bridge_width 0.5)
+			(island_removal_mode 0)
+		)
+		(polygon
+			(pts
+				(xy 63.5 29.5) (xy 139 29.5) (xy 139 101.5) (xy 63.5 101.5)
+			)
+		)
+	)
+	(zone
+		(net "GND")
+		(layer "B.Cu")
+		(hatch edge 0.5)
+		(priority 1)
+		(connect_pads
+			(clearance 0.5)
+		)
+		(min_thickness 0.25)
+		(fill yes
+			(thermal_gap 0.5)
+			(thermal_bridge_width 0.5)
+			(island_removal_mode 0)
+		)
+		(polygon
+			(pts
+				(xy 63.5 29.5) (xy 139 29.5) (xy 139 101.5) (xy 63.5 101.5)
+			)
+		)
+	)
 	(embedded_fonts no)
